File: 02-vco/electronics/core-2layer/vco-core.kicad_pcb (KiCad board)
At the start: 2 copper layers, 48 x 110 mm, 112 parts, among them J1 Conn_01x04, J2 Conn_02x05_Odd_Even, J3 Conn_02x05_Odd_Even, J5 Conn_02x03_Odd_Even, Q1 BC847BS, Q2 MMBT3906, Q3 J111, Q4 MMBFJ111, Q5 MMBT5551, U1 TL072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

Commit message: Cleanup
Parts:
- moved ? 14.9 mm to (146.7, 152.4)
Changed lines of the file:
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@@
 		(locked yes)
 		(layer "F.Cu")
-		(at 131.826 152.527)
+		(at 146.685 152.4)
 		(property "Reference" ""
 			(at 0 0 0)
@@
 	)
 	(gr_text "Trace sizes:\nSignal — 20mil\nPower — 35mil"
-		(at 149.479 34.798 0)
+		(at 123.571 33.782 0)
 		(layer "User.2")
 		(effects
@@
 			(keep_text_aligned yes)
 		)
-		(gr_text "4094.4882"
+		(gr_text "104"
 			(at 94.85 96 90)
 			(layer "User.2")
@@
 			(keep_text_aligned yes)
 		)
-		(gr_text "590.5512"
+		(gr_text "15"
 			(locked yes)
 			(at 111.85 96.5 90)
@@
 			(keep_text_aligned yes)
 		)
-		(gr_text "354.3307"
+		(gr_text "9"
 			(locked yes)
 			(at 111.85 149.5 90)
@@
 			(keep_text_aligned yes)
 		)
-		(gr_text "1889.7638"
+		(gr_text "48"
 			(at 148 38.85 0)
 			(layer "User.2")
@@
 			(keep_text_aligned yes)
 		)
-		(gr_text "2204.7244"
+		(gr_text "56"
 			(at 100.35 72 90)
 			(layer "User.2")
@@
 			(keep_text_aligned yes)
 		)
-		(gr_text "1948.8189"
+		(gr_text "49.5"
 			(at 105.85 68.75 90)
 			(layer "User.2")
@@
 			(keep_text_aligned yes)
 		)
-		(gr_text "1771.6535"
+		(gr_text "45"
 			(locked yes)
 			(at 111.85 66.5 90)
@@
 			(keep_text_aligned yes)
 		)
-		(gr_text "2165.3543"
+		(gr_text "55"
 			(at 176.85 71.5 90)
 			(layer "User.2")
@@
 			(keep_text_aligned yes)
 		)
-		(gr_text "1614.1732"
+		(gr_text "41"
 			(locked yes)
 			(at 111.85 124.5 90)
