File: 02-vco/electronics/core/sheets/raw-oscillator.kicad_sch (KiCad schematic)
At the start: 56 parts, among them Q1 BC847BS, Q2 2N3906, Q3 J111, Q4 MMBFJ111, Q5 MMBT5551, U1 TL072, U2 TL072, U3 LM311

Commit message: Designed VCO core PCB
Parts:
- Q1: LCSC (none) -> C5380687; Vendor (none) -> JLCPCB
- Q2: value 2N3906 -> MMBT3906; footprint Package_TO_SOT_THT:TO-92_Inline -> Package_TO_SOT_SMD:SOT-23_Handsoldering; LCSC (none) -> C7420354; Vendor (none) -> JLCPCB
- renumbered R_HIFREQ1 to R_BIAS1, R_HIFREQ2 to R_HIFREQ1
Other:
- moved on the sheet: C1, C10, C11, C2, C3, C4, C5, C6, C7, C8, C9, D1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

Commit message: Refined VCO core and UI
Parts:
- C1, C10, C11, C2, C3, C4, C5, C6, C8, D1, Q4, Q5, R1, R10, R11, R12, R13, R14, R15, R16, R17, R18, R19, R2, R20, R21, R22, R4, R5, R9, U1, U2, U3: CHECKED (none) -> YES; Vendor (none) -> JLCPCB
- C7: CHECKED (none) -> YES; now not fitted
- C9: CHECKED (none) -> YES; Mouser Part no. (none) -> 80-R82MC1220AA50J; Part URL (none) -> https://mou.sr/4eLPHe3; Vendor (none) -> Mouser; now in the parts list
- Q1, Q2, TP1, TP2, TP3, TP4, TP5: CHECKED (none) -> YES
- Q3: CHECKED (none) -> YES; Mouser 512-J111 -> (none); Mouser Part no. (none) -> 512-J111; Part URL (none) -> https://mou.sr/4f5W0HS; Vendor (none) -> Mouser; now in the parts list
- R3, R6, R7: CHECKED (none) -> YES; now in the parts list
- R8: CHECKED (none) -> YES; Mouser https://hu.mouser.com/ProductDetail/YAGEO/MFR50SFTE52-4R22?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 -> (none); Part URL (none) -> https://hu.mouser.com/ProductDetail/YAGEO/MFR50SFTE52-4R22?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; now in the parts list
- R_BIAS1: CHECKED (none) -> YES; Mouser Part no. (none) -> 652-3006P-1-104-LF; Part URL (none) -> https://mou.sr/4ff5W1E; Vendor (none) -> Mouser; now in the parts list
- R_HIFREQ1: CHECKED (none) -> YES; Mouser Part no. (none) -> 652-3006P-1-202-LF; Part URL (none) -> https://mou.sr/3ZK9AMt; Vendor (none) -> Mouser; now in the parts list
- R_WIDTH1: CHECKED (none) -> YES; Mouser Part no. (none) -> 652-3006P-7-203-LF; Part URL (none) -> https://mou.sr/41re1x3; Vendor (none) -> Mouser; now in the parts list
- R_WIDTH2: CHECKED (none) -> YES; Mouser Part no. (none) -> 652-3006P-1-501-LF; Part URL (none) -> https://mou.sr/3GyUiUc; Vendor (none) -> Mouser; now in the parts list
- TH1: CHECKED (none) -> YES; Mouser Part no. (none) -> 594-2381-640-55103; Part URL (none) -> https://mou.sr/4nM5nSy; Vendor (none) -> Mouser; now in the parts list
- TH2: CHECKED (none) -> YES; Mouser https://hu.mouser.com/ProductDetail/594-PTS120601B100RP -> (none); Mouser Part no. (none) -> 594-PTS120601B100RP; Part URL (none) -> https://hu.mouser.com/ProductDetail/594-PTS120601B100RP; Vendor (none) -> Mouser; now in the parts list
