File: 04-vcf/electronics/core/vcf.kicad_pcb (KiCad board)
At the start: 2 copper layers, 58 x 110 mm, 84 parts, among them J1 Conn_01x06, J2 Conn_02x05_Odd_Even, J3 Conn_02x02_Counter_Clockwise, J4 S1711-46R, J5 S1711-46R, J6 Conn_02x03_Odd_Even, J7 Conn_01x02, J8 Conn_02x05_Odd_Even, Q1 BC847BS, U1 TL072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

Commit message: Finished v0.1 of VCF PCB
Parts:
- added G***: LOGO, Shmoergh_Custom_Footprints:Gyeszno, F.Cu at (127.6, 125.0)
- added G***: LOGO, Shmoergh_Logo:Gyeszno, F.Cu at (128.3, 109.0)
- added G***: LOGO, Shmoergh_Logo:Gyeszno, B.Cu at (137.0, 108.3)
- added G***: LOGO, Shmoergh_Custom_Footprints:Gyeszno, B.Cu at (152.4, 98.6)
- added G***: LOGO, Shmoergh_Custom_Footprints:Gyeszno, B.Cu at (174.2, 136.5)
- J2: value Conn_02x05_Odd_Even -> Conn_02x04_Counter_Clockwise; footprint Connector_PinHeader_2.54mm:PinHeader_2x05_P2.54mm_Vertical -> Connector_PinHeader_2.54mm:PinHeader_2x04_P2.54mm_Vertical
- R15: value 33k -> 33k?
- moved R24 129.2 mm to (139.0, 145.1), turned to -90 degrees
- moved R25 128.9 mm to (137.4, 145.1), turned to -90 degrees
- moved R26 128.7 mm to (135.7, 145.1), turned to 90 degrees
- moved TP2 124.6 mm to (169.2, 140.3)
- moved C11 124.2 mm to (127.8, 132.6)
- moved R29 115.3 mm to (139.1, 133.8), turned to 90 degrees
- moved R32 114.6 mm to (135.8, 133.8), turned to -90 degrees
- moved R31 114.3 mm to (137.5, 133.8), turned to 90 degrees
- moved J3 111.4 mm to (170.0, 148.5)
- moved C5 110.8 mm to (134.1, 135.3), turned to 90 degrees
- moved C19 109.4 mm to (130.3, 137.0), turned to -90 degrees
- moved C6 108.6 mm to (140.9, 143.4), turned to 90 degrees
- moved R17 107.1 mm to (155.0, 142.4)
- moved C18 105.9 mm to (144.3, 142.0), turned to 90 degrees
- moved J7 104.5 mm to (151.8, 92.5), turned to 90 degrees
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Connections:
- J2 pad 1: LP -> GND
- J2 pad 2: GND -> OUT
- J2 pad 3: HP -> LP
- J2 pad 5: CUTOFF -> HP
- J2 pad 7: OUT -> CUTOFF
- J3 pad 1: RESO_IN -> RESO_OUT
- J3 pad 3: RESO_OUT -> RESO_IN
Routing:
- net -12V: track 36.0 -> 149.4 mm, vias 0 -> 4
- net +12V: track 63.8 -> 163.3 mm, vias 0 -> 2
- net CUTOFF: track 4.13 -> 67.0 mm, vias 0 -> 2
- net Net-(C11-Pad1): track 0.00 -> 56.1 mm, vias 0 -> 4
- net Net-(D1-K): track 0.00 -> 51.5 mm
- net Net-(C19-Pad2): track 0.00 -> 45.3 mm
- net Net-(C10-Pad2): track 3.17 -> 46.4 mm, vias 0 -> 4
- net Net-(Q1A-B1): track 3.85 -> 43.7 mm, vias 0 -> 4
- net HP: track 0.00 -> 39.4 mm
- net OUT: track 0.00 -> 38.7 mm
- net RESO_OUT: track 0.00 -> 38.1 mm
- net Net-(D10-A): track 8.89 -> 41.5 mm
- net Net-(C11-Pad2): track 1.65 -> 33.0 mm, vias 0 -> 4
- net Net-(C12-Pad2): track 2.62 -> 30.0 mm, vias 0 -> 2
- net LP: track 0.00 -> 27.2 mm
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- added copper zone on F.Cu, net GND
Other:
- board size 58 x 110 mm -> 58 x 65 mm
- board text added: "-12V"
- board text added: "BALANCE"
- board text added: "CO1"
- board text added: "CO2"
- board text added: "CUT"
- board text added: "DEFAULTS"
- board text added: "HM-04 Diode Filter V0.1 2025 July"
- board text added: "HP"
- board text added: "LP"
- board text added: "MAX RESO"
- board text added: "NC"
- board text added: "OUT"
- board text added: "POWER"
- board text added: "SHMØERGH HOG MODULEUR"
- board text added: "TP:+12V"
- board text added: "TP:-12V"
- board text added: "TP:2xGND"
