File: 03-sidechain-mixer/electronics/core/sidechain-mixer-core.kicad_pcb (KiCad board)
At the start: 2 copper layers, 58 x 65 mm, 70 parts, among them J1 Conn_02x04_Odd_Even, J2 Conn_02x05_Odd_Even, J3 Conn_02x05_Odd_Even, J4 Conn_01x02, J5 Conn_02x03_Odd_Even, J8 Conn_01x06, Q1 BC847BS, U1 TL072, U2 TL072, U3 TL072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

Commit message: Added SC Mixer UI schematics
Parts:
- added REF**: ToolingHole_1.152mm, MountingHole:ToolingHole_1.152mm, F.Cu at (125.1, 96.2)
- added REF**: ToolingHole_1.152mm, MountingHole:ToolingHole_1.152mm, F.Cu at (130.0, 147.0)
- added REF**: ToolingHole_1.152mm, MountingHole:ToolingHole_1.152mm, F.Cu at (180.4, 146.0)
- R18, R19, R26, R28: value 100k -> 10k
Routing:
- net GND: vias 322 -> 319

Commit message: Sidechain Mixer UI PCB RC
Parts:
- added J6: Conn_01x04, Connector_PinHeader_2.54mm:PinHeader_1x04_P2.54mm_Vertical, F.Cu at (145.0, 98.5)
- J1: value Conn_02x04_Odd_Even -> Conn_01x04; footprint Connector_PinHeader_2.54mm:PinHeader_2x04_P2.54mm_Vertical -> Connector_PinHeader_2.54mm:PinHeader_1x04_P2.54mm_Vertical
- moved J5 49.5 mm to (150.5, 151.0)
- moved G*** 43.3 mm to (133.9, 101.4)
- moved J1 10.0 mm to (126.0, 107.5), turned to 0 degrees
- moved G*** 2.27 mm to (148.5, 112.2)
- moved R26 0.46 mm to (155.5, 141.6)
- moved R18 0.36 mm to (152.4, 141.6)
Connections:
- J1 pad 1: MAIN_VOL_3 -> MAIN_VOL_1
- J1 pad 2: MAIN_VOL_1 -> CH_4_VOL_2
- J1 pad 3: RATIO_1 -> CH_4_GAIN_1
- J1 pad 4: CH_4_VOL_2 -> CH_4_GAIN_3_VOL_3
Routing:
- net CH_4_GAIN_1: track 74.4 -> 41.3 mm
- net CH_4_GAIN_3_VOL_3: track 82.0 -> 50.4 mm
- net CH_4_VOL_2: track 32.1 -> 11.9 mm
- net MAIN_VOL_1: track 40.5 -> 30.1 mm
- net +12V: track 154.9 -> 161.7 mm, vias 4 -> 5
- net THRESHOLD: track 47.4 -> 41.1 mm
- net RATIO_3: track 64.5 -> 58.5 mm
- net -12V: track 134.9 -> 139.4 mm, vias 2 -> 4
- net RATIO_1: track 71.6 -> 67.6 mm
- net Net-(U3B--): track 57.9 -> 58.8 mm
- net Net-(U4B-+): track 22.1 -> 22.9 mm
- net GND: vias 319 -> 347
Other:
- board text added: "CH_4_GAIN_1"
- board text added: "CH_4_GAIN_3_VOL_3"
- board text added: "CH_4_VOL_2"
- board text added: "GND"
- board text added: "MAIN_VOL_1"
- board text added: "MAIN_VOL_3"
- board text removed: "5xGND"
- board text removed: "CH4_1"
- board text removed: "CH4_3"
- board text removed: "M_V_3"
- board text removed: "RAT_1"
- board text removed: "RAT_3"
- board text removed: "THRS"

Commit message: Checked all components on SC-Mixer
Parts:
- D1, D2: footprint Diode_SMD:D_SOD-323_HandSoldering -> Diode_SMD:D_SOD-123
- moved D1 0.25 mm to (173.9, 135.9)
- moved D2 0.13 mm to (133.0, 136.2)
Other:
- board text added: "+"
