File: 05-adsr-vca/electronics/v0.2/ui/adsr-vca-ui.kicad_sch (KiCad schematic)
At the start: 23 parts, among them J1 Conn_02x03_Odd_Even, J3 Conn_02x03_Odd_Even, J4 Conn_01x02, J5 Conn_01x06, J6 Conn_02x03_Odd_Even, J8 Conn_02x03_Odd_Even

Commit message: Redraw ADSR PCBs to be on top half of the UI
Connections:
- net ATTACK_3: now also J8.2 (Pin_2); no longer J8.4 (Pin_4)
- net DECAY_1: now also J8.5 (Pin_5); no longer J8.2 (Pin_2)
- net ENV_OUT: now also J8.4 (Pin_4); no longer J8.3 (Pin_3)
- net RELEASE_1: now also J8.3 (Pin_3)
- no-connect marks 6 -> 5
Other:
- moved on the sheet: D1, J3, J5, J6, J8
