File: 05-adsr-vca/electronics/core/sheets/power.kicad_sch (KiCad schematic)
At the start: 7 parts, among them J3 Conn_02x05_Odd_Even, J4 Conn_01x02, J5 Conn_02x03_Odd_Even

Commit message: VCA PCB WIP
Parts:
- C10: renamed from C24; CHECKED YES -> (none)
- C9: renamed from C23; CHECKED YES -> (none)
- D4: renamed from D6; CHECKED YES -> (none)
- D5: renamed from D7; CHECKED YES -> (none)
- renumbered J4 to J6, J3 to J7
Changed lines of the file:
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@@
 		(dnp no)
 		(fields_autoplaced yes)
-		(property "Reference" "#PWR059"
+		(property "Reference" "#PWR028"
 			(at 104.14 87.63 0)
 			(effects
@@
 			(project "vco-core"
 				(path "/8e2e31f3-eed5-4de1-966c-f4162758c735/8bc1c38c-66cf-4d37-87f2-6eda8e5acaa7"
-					(reference "#PWR059")
+					(reference "#PWR028")
 					(unit 1)
 				)
@@
 		(dnp no)
 		(fields_autoplaced yes)
-		(property "Reference" "C23"
+		(property "Reference" "C9"
 			(at 234.95 89.281 0)
 			(effects
@@
 			)
 		)
-		(property "CHECKED" "YES"
+		(property "CHECKED" ""
 			(at 231.14 91.44 0)
 			(effects
@@
 			(project "vco-core"
 				(path "/8e2e31f3-eed5-4de1-966c-f4162758c735/8bc1c38c-66cf-4d37-87f2-6eda8e5acaa7"
-					(reference "C23")
+					(reference "C9")
 					(unit 1)
 				)
@@
 		(dnp no)
 		(fields_autoplaced yes)
-		(property "Reference" "#PWR047"
+		(property "Reference" "#PWR030"
 			(at 137.16 115.57 0)
 			(effects
@@
 			(project ""
 				(path "/8e2e31f3-eed5-4de1-966c-f4162758c735/8bc1c38c-66cf-4d37-87f2-6eda8e5acaa7"
-					(reference "#PWR047")
+					(reference "#PWR030")
 					(unit 1)
 				)
@@
 		(on_board yes)
 		(dnp no)
-		(property "Reference" "D7"
+		(property "Reference" "D5"
 			(at 175.26 109.22 0)
 			(effects
@@
 			)
 		)
-		(property "CHECKED" "YES"
+		(property "CHECKED" ""
 			(at 175.26 106.68 0)
 			(effects
@@
 			(project "vco-core"
 				(path "/8e2e31f3-eed5-4de1-966c-f4162758c735/8bc1c38c-66cf-4d37-87f2-6eda8e5acaa7"
-					(reference "D7")
+					(reference "D5")
 					(unit 1)
 				)
@@
 		(dnp no)
 		(fields_autoplaced yes)
-		(property "Reference" "#PWR050"
+		(property "Reference" "#PWR032"
 			(at 181.61 105.41 0)
 			(effects
@@
 			(project "vco-core"
 				(path "/8e2e31f3-eed5-4de1-966c-f4162758c735/8bc1c38c-66cf-4d37-87f2-6eda8e5acaa7"
-					(reference "#PWR050")
+					(reference "#PWR032")
 					(unit 1)
 				)
@@
 		(dnp no)
 		(fields_autoplaced yes)
-		(property "Reference" "#PWR060"
+		(property "Reference" "#PWR026"
 			(at 77.47 93.98 0)
 			(effects
@@
 			(project "vco-core"
 				(path "/8e2e31f3-eed5-4de1-966c-f4162758c735/8bc1c38c-66cf-4d37-87f2-6eda8e5acaa7"
-					(reference "#PWR060")
+					(reference "#PWR026")
 					(unit 1)
 				)
@@
 		(dnp no)
 		(fields_autoplaced yes)
-		(property "Reference" "#PWR052"
+		(property "Reference" "#PWR034"
 			(at 226.06 110.49 0)
 			(effects
@@
 			(project "vco-core"
 				(path "/8e2e31f3-eed5-4de1-966c-f4162758c735/8bc1c38c-66cf-4d37-87f2-6eda8e5acaa7"
-					(reference "#PWR052")
+					(reference "#PWR034")
 					(unit 1)
 				)
@@
 		(dnp no)
 		(fields_autoplaced yes)
-		(property "Reference" "#PWR049"
+		(property "Reference" "#PWR033"
 			(at 181.61 105.41 0)
 			(effects
@@
 			(project ""
 				(path "/8e2e31f3-eed5-4de1-966c-f4162758c735/8bc1c38c-66cf-4d37-87f2-6eda8e5acaa7"
-					(reference "#PWR049")
+					(reference "#PWR033")
 					(unit 1)
 				)
@@
 		(dnp no)
 		(fields_autoplaced yes)
-		(property "Reference" "C24"
+		(property "Reference" "C10"
 			(at 234.95 96.901 0)
 			(effects
@@
 			)
 		)
-		(property "CHECKED" "YES"
+		(property "CHECKED" ""
 			(at 231.14 99.06 0)
 			(effects
@@
 			(project "vco-core"
 				(path "/8e2e31f3-eed5-4de1-966c-f4162758c735/8bc1c38c-66cf-4d37-87f2-6eda8e5acaa7"
-					(reference "C24")
+					(reference "C10")
 					(unit 1)
 				)
@@
 		(dnp no)
 		(fields_autoplaced yes)
-		(property "Reference" "#PWR061"
+		(property "Reference" "#PWR025"
 			(at 71.12 104.14 0)
 			(effects
@@
 			(project "vco-core"
 				(path "/8e2e31f3-eed5-4de1-966c-f4162758c735/8bc1c38c-66cf-4d37-87f2-6eda8e5acaa7"
-					(reference "#PWR061")
+					(reference "#PWR025")
 					(unit 1)
 				)
@@
 		(on_board yes)
 		(dnp no)
-		(property "Reference" "J3"
+		(property "Reference" "J7"
 			(at 154.94 86.36 0)
 			(effects
@@
 			(project ""
 				(path "/8e2e31f3-eed5-4de1-966c-f4162758c735/8bc1c38c-66cf-4d37-87f2-6eda8e5acaa7"
-					(reference "J3")
+					(reference "J7")
 					(unit 1)
 				)
@@
 		(dnp no)
 		(fields_autoplaced yes)
-		(property "Reference" "#PWR053"
+		(property "Reference" "#PWR035"
 			(at 231.14 90.17 0)
 			(effects
@@
 			(project "vco-core"
 				(path "/8e2e31f3-eed5-4de1-966c-f4162758c735/8bc1c38c-66cf-4d37-87f2-6eda8e5acaa7"
-					(reference "#PWR053")
+					(reference "#PWR035")
 					(unit 1)
 				)
@@
 		(on_board yes)
 		(dnp no)
-		(property "Reference" "D6"
+		(property "Reference" "D4"
 			(at 173.99 80.01 0)
 			(effects
@@
 			)
 		)
-		(property "CHECKED" "YES"
+		(property "CHECKED" ""
 			(at 173.99 85.09 0)
 			(effects
@@
 			(project ""
 				(path "/8e2e31f3-eed5-4de1-966c-f4162758c735/8bc1c38c-66cf-4d37-87f2-6eda8e5acaa7"
-					(reference "D6")
+					(reference "D4")
 					(unit 1)
 				)
@@
 		(dnp no)
 		(fields_autoplaced yes)
-		(property "Reference" "#PWR048"
+		(property "Reference" "#PWR031"
 			(at 180.34 86.36 0)
 			(effects
@@
 			(project ""
 				(path "/8e2e31f3-eed5-4de1-966c-f4162758c735/8bc1c38c-66cf-4d37-87f2-6eda8e5acaa7"
-					(reference "#PWR048")
+					(reference "#PWR031")
 					(unit 1)
 				)
@@
 		(dnp no)
 		(fields_autoplaced yes)
-		(property "Reference" "J4"
+		(property "Reference" "J6"
 			(at 95.25 109.2199 0)
 			(effects
@@
 			(project ""
 				(path "/8e2e31f3-eed5-4de1-966c-f4162758c735/8bc1c38c-66cf-4d37-87f2-6eda8e5acaa7"
-					(reference "J4")
+					(reference "J6")
 					(unit 1)
 				)
@@
 		(dnp no)
 		(fields_autoplaced yes)
-		(property "Reference" "#PWR058"
+		(property "Reference" "#PWR027"
 			(at 85.09 119.38 0)
 			(effects
@@
 			(project "vco-core"
 				(path "/8e2e31f3-eed5-4de1-966c-f4162758c735/8bc1c38c-66cf-4d37-87f2-6eda8e5acaa7"
-					(reference "#PWR058")
+					(reference "#PWR027")
 					(unit 1)
 				)
@@
 		(dnp no)
 		(fields_autoplaced yes)
-		(property "Reference" "#PWR054"
+		(property "Reference" "#PWR036"
 			(at 231.14 106.68 0)
 			(effects
@@
 			(project "vco-core"
 				(path "/8e2e31f3-eed5-4de1-966c-f4162758c735/8bc1c38c-66cf-4d37-87f2-6eda8e5acaa7"
-					(reference "#PWR054")
+					(reference "#PWR036")
 					(unit 1)
 				)
@@
 		(dnp no)
 		(fields_autoplaced yes)
-		(property "Reference" "#PWR062"
+		(property "Reference" "#PWR029"
 			(at 104.14 104.14 0)
 			(effects
@@
 			(project "vco-core"
 				(path "/8e2e31f3-eed5-4de1-966c-f4162758c735/8bc1c38c-66cf-4d37-87f2-6eda8e5acaa7"
-					(reference "#PWR062")
-					(unit 1)
-				)
+					(reference "#PWR029")
+					(unit 1)
+				)

Commit message: ADSR+VCA production files ready
Parts:
- C10, C9, D4, D5: CHECKED (none) -> YES
Changed lines of the file:
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@@
 			)
 		)
-		(property "CHECKED" ""
+		(property "CHECKED" "YES"
 			(at 231.14 91.44 0)
 			(effects
@@
 			)
 		)
-		(property "CHECKED" ""
+		(property "CHECKED" "YES"
 			(at 175.26 106.68 0)
 			(effects
@@
 			)
 		)
-		(property "CHECKED" ""
+		(property "CHECKED" "YES"
 			(at 231.14 99.06 0)
 			(effects
@@
 			)
 		)
-		(property "CHECKED" ""
+		(property "CHECKED" "YES"
 			(at 173.99 85.09 0)
 			(effects
