File: 06-utils-output/electronics/core/sheets/output.kicad_sch (KiCad schematic)
At the start: 30 parts, among them U4 NE5532, U5 TL072

Commit message: Fixed Release pot polarity
Parts:
- renumbered D13 to #D13, D14 to #D14
Changed lines of the file:
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@@
 		(on_board yes)
 		(dnp no)
-		(property "Reference" "D14"
+		(property "Reference" "#D14"
 			(at 71.12 66.04 90)
 			(effects
@@
 			(project "utils-output-core"
 				(path "/8e2e31f3-eed5-4de1-966c-f4162758c735/41496549-080e-47b7-9088-5316bbc20ed8"
-					(reference "D14")
+					(reference "#D14")
 					(unit 1)
 				)
@@
 		(on_board yes)
 		(dnp no)
-		(property "Reference" "D13"
+		(property "Reference" "#D13"
 			(at 71.12 54.61 90)
 			(effects
@@
 			(project "utils-output-core"
 				(path "/8e2e31f3-eed5-4de1-966c-f4162758c735/41496549-080e-47b7-9088-5316bbc20ed8"
-					(reference "D13")
+					(reference "#D13")
 					(unit 1)
 				)

Commit message: Utils+output PCB v0.1 ready
Parts:
- removed D17: SMAJ5.0CA, Diode_SMD:D_SMA, symbol Diode:SMAJ5.0CA
- C10, C11, C12, C13, C15, D15, D16, D_LIM_N1, D_LIM_P1, R11, R12, R13, R14, R15, R25, RV_HEADPHONE_LIM1, RV_LINE_OUT_LVL1, TP1, TP2, TP3, U4, U5: CHECKED (none) -> YES
- C14: footprint Capacitor_THT:CP_Radial_D5.0mm_P2.00mm -> Capacitor_SMD:CP_Elec_5x5.4; CHECKED (none) -> YES; LCSC (none) -> C4747971; Vendor (none) -> JLCPCB
- R24: CHECKED (none) -> YES; LCSC (none) -> C31850
- R29: CHECKED (none) -> YES; LCSC C21190 -> C25804
Other:
- note removed: "?????"
- moved on the sheet: R14, R15, RV_HEADPHONE_LIM1, TP3, U4A, U4B
