File: 07-brain/electronics/ui/sheets/leds.kicad_sch (KiCad schematic)
At the start: 24 parts, among them Q1 2N3904, Q2 2N3904, Q3 2N3904, Q4 2N3904, Q5 2N3904, Q6 2N3904

Commit message: Designed Brain UI PCB
Connections:
- net at D3.2 (A): now also R13.1; no longer R9.1
- net at D4.2 (A): now also R6.1; no longer R10.1
- net at Q5.2 (B): now also R8.2; no longer R11.2
- net at Q4.2 (B): now also R4.2; no longer R8.2
- net at Q2.2 (B): now also R7.2; no longer R4.2
- net at D5.2 (A): now also R10.1; no longer R13.1
- net at Q3.2 (B): now also R11.2; no longer R7.2
- net at D2.2 (A): now also R9.1; no longer R6.1
Other:
- moved on the sheet: D2, D3, D4, D5, Q2, Q3, Q4, Q5
Changed lines of the file:
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@@
 	(symbol
 		(lib_id "Device:LED")
-		(at 154.94 55.88 90)
+		(at 218.44 55.88 90)
 		(unit 1)
 		(exclude_from_sim no)
@@
 		(fields_autoplaced yes)
 		(property "Reference" "D3"
-			(at 158.75 56.1974 90)
+			(at 222.25 56.1974 90)
 			(effects
 				(font
@@
 		)
 		(property "Value" "LED"
-			(at 158.75 58.7374 90)
+			(at 222.25 58.7374 90)
 			(effects
 				(font
@@
 		)
 		(property "Footprint" "LED_THT:LED_D3.0mm"
-			(at 154.94 55.88 0)
+			(at 218.44 55.88 0)
 			(effects
 				(font
@@
 		)
 		(property "Datasheet" "~"
-			(at 154.94 55.88 0)
+			(at 218.44 55.88 0)
 			(effects
 				(font
@@
 		)
 		(property "Description" "Light emitting diode"
-			(at 154.94 55.88 0)
+			(at 218.44 55.88 0)
 			(effects
 				(font
@@
 		)
 		(property "Sim.Pins" "1=K 2=A"
-			(at 154.94 55.88 0)
+			(at 218.44 55.88 0)
 			(effects
 				(font
@@
 	(symbol
 		(lib_id "Device:LED")
-		(at 154.94 119.38 90)
+		(at 91.44 119.38 90)
 		(unit 1)
 		(exclude_from_sim no)
@@
 		(fields_autoplaced yes)
 		(property "Reference" "D4"
-			(at 158.75 119.6974 90)
+			(at 95.25 119.6974 90)
 			(effects
 				(font
@@
 		)
 		(property "Value" "LED"
-			(at 158.75 122.2374 90)
+			(at 95.25 122.2374 90)
 			(effects
 				(font
@@
 		)
 		(property "Footprint" "LED_THT:LED_D3.0mm"
-			(at 154.94 119.38 0)
+			(at 91.44 119.38 0)
 			(effects
 				(font
@@
 		)
 		(property "Datasheet" "~"
-			(at 154.94 119.38 0)
+			(at 91.44 119.38 0)
 			(effects
 				(font
@@
 		)
 		(property "Description" "Light emitting diode"
-			(at 154.94 119.38 0)
+			(at 91.44 119.38 0)
 			(effects
 				(font
@@
 		)
 		(property "Sim.Pins" "1=K 2=A"
-			(at 154.94 119.38 0)
+			(at 91.44 119.38 0)
 			(effects
 				(font
@@
 	(symbol
 		(lib_id "Transistor_BJT:2N3904")
-		(at 215.9 67.31 0)
+		(at 152.4 130.81 0)
 		(unit 1)
 		(exclude_from_sim no)
@@
 		(fields_autoplaced yes)
 		(property "Reference" "Q5"
-			(at 220.98 66.0399 0)
+			(at 157.48 129.5399 0)
 			(effects
 				(font
@@
 		)
 		(property "Value" "2N3904"
-			(at 220.98 68.5799 0)
+			(at 157.48 132.0799 0)
 			(effects
 				(font
@@
 		)
 		(property "Footprint" "Package_TO_SOT_THT:TO-92_Inline_Wide"
-			(at 220.98 69.215 0)
+			(at 157.48 132.715 0)
 			(effects
 				(font
@@
 		)
 		(property "Datasheet" "https://www.onsemi.com/pub/Collateral/2N3903-D.PDF"
-			(at 215.9 67.31 0)
+			(at 152.4 130.81 0)
 			(effects
 				(font
@@
 		)
 		(property "Description" "0.2A Ic, 40V Vce, Small Signal NPN Transistor, TO-92"
-			(at 215.9 67.31 0)
+			(at 152.4 130.81 0)
 			(effects
 				(font
@@
 	(symbol
 		(lib_id "Transistor_BJT:2N3904")
-		(at 152.4 130.81 0)
+		(at 88.9 130.81 0)
 		(unit 1)
 		(exclude_from_sim no)
@@
 		(fields_autoplaced yes)
 		(property "Reference" "Q4"
-			(at 157.48 129.5399 0)
+			(at 93.98 129.5399 0)
 			(effects
 				(font
@@
 		)
 		(property "Value" "2N3904"
-			(at 157.48 132.0799 0)
+			(at 93.98 132.0799 0)
 			(effects
 				(font
@@
 		)
 		(property "Footprint" "Package_TO_SOT_THT:TO-92_Inline_Wide"
-			(at 157.48 132.715 0)
+			(at 93.98 132.715 0)
 			(effects
 				(font
@@
 		)
 		(property "Datasheet" "https://www.onsemi.com/pub/Collateral/2N3903-D.PDF"
-			(at 152.4 130.81 0)
+			(at 88.9 130.81 0)
 			(effects
 				(font
@@
 		)
 		(property "Description" "0.2A Ic, 40V Vce, Small Signal NPN Transistor, TO-92"
-			(at 152.4 130.81 0)
+			(at 88.9 130.81 0)
 			(effects
 				(font
@@
 	(symbol
 		(lib_id "Device:LED")
-		(at 218.44 55.88 90)
+		(at 154.94 119.38 90)
 		(unit 1)
 		(exclude_from_sim no)
@@
 		(fields_autoplaced yes)
 		(property "Reference" "D5"
-			(at 222.25 56.1974 90)
+			(at 158.75 119.6974 90)
 			(effects
 				(font
@@
 		)
 		(property "Value" "LED"
-			(at 222.25 58.7374 90)
+			(at 158.75 122.2374 90)
 			(effects
 				(font
@@
 		)
 		(property "Footprint" "LED_THT:LED_D3.0mm"
-			(at 218.44 55.88 0)
+			(at 154.94 119.38 0)
 			(effects
 				(font
@@
 		)
 		(property "Datasheet" "~"
-			(at 218.44 55.88 0)
+			(at 154.94 119.38 0)
 			(effects
 				(font
@@
 		)
 		(property "Description" "Light emitting diode"
-			(at 218.44 55.88 0)
+			(at 154.94 119.38 0)
 			(effects
 				(font
@@
 		)
 		(property "Sim.Pins" "1=K 2=A"
-			(at 218.44 55.88 0)
+			(at 154.94 119.38 0)
 			(effects
 				(font
@@
 	(symbol
 		(lib_id "Transistor_BJT:2N3904")
-		(at 88.9 130.81 0)
+		(at 152.4 67.31 0)
 		(unit 1)
 		(exclude_from_sim no)
@@
 		(fields_autoplaced yes)
 		(property "Reference" "Q2"
-			(at 93.98 129.5399 0)
+			(at 157.48 66.0399 0)
 			(effects
 				(font
@@
 		)
 		(property "Value" "2N3904"
-			(at 93.98 132.0799 0)
+			(at 157.48 68.5799 0)
 			(effects
 				(font
@@
 		)
 		(property "Footprint" "Package_TO_SOT_THT:TO-92_Inline_Wide"
-			(at 93.98 132.715 0)
+			(at 157.48 69.215 0)
 			(effects
 				(font
@@
 		)
 		(property "Datasheet" "https://www.onsemi.com/pub/Collateral/2N3903-D.PDF"
-			(at 88.9 130.81 0)
+			(at 152.4 67.31 0)
 			(effects
 				(font
@@
 		)
 		(property "Description" "0.2A Ic, 40V Vce, Small Signal NPN Transistor, TO-92"
-			(at 88.9 130.81 0)
+			(at 152.4 67.31 0)
 			(effects
 				(font
@@
 	(symbol
 		(lib_id "Device:LED")
-		(at 91.44 119.38 90)
+		(at 154.94 55.88 90)
 		(unit 1)
 		(exclude_from_sim no)
@@
 		(fields_autoplaced yes)
 		(property "Reference" "D2"
-			(at 95.25 119.6974 90)
+			(at 158.75 56.1974 90)
 			(effects
 				(font
@@
 		)
 		(property "Value" "LED"
-			(at 95.25 122.2374 90)
+			(at 158.75 58.7374 90)
 			(effects
 				(font
@@
 		)
 		(property "Footprint" "LED_THT:LED_D3.0mm"
-			(at 91.44 119.38 0)
+			(at 154.94 55.88 0)
 			(effects
 				(font
@@
 		)
 		(property "Datasheet" "~"
-			(at 91.44 119.38 0)
+			(at 154.94 55.88 0)
 			(effects
 				(font
@@
 		)
 		(property "Description" "Light emitting diode"
-			(at 91.44 119.38 0)
+			(at 154.94 55.88 0)
 			(effects
 				(font
@@
 		)
 		(property "Sim.Pins" "1=K 2=A"
-			(at 91.44 119.38 0)
+			(at 154.94 55.88 0)
 			(effects
 				(font
@@
 	(symbol
 		(lib_id "Transistor_BJT:2N3904")
-		(at 152.4 67.31 0)
+		(at 215.9 67.31 0)
 		(unit 1)
 		(exclude_from_sim no)
@@
 		(fields_autoplaced yes)
 		(property "Reference" "Q3"
-			(at 157.48 66.0399 0)
+			(at 220.98 66.0399 0)
 			(effects
 				(font
@@
 		)
 		(property "Value" "2N3904"
-			(at 157.48 68.5799 0)
+			(at 220.98 68.5799 0)
 			(effects
 				(font
@@
 		)
 		(property "Footprint" "Package_TO_SOT_THT:TO-92_Inline_Wide"
-			(at 157.48 69.215 0)
+			(at 220.98 69.215 0)
 			(effects
 				(font
@@
 		)
 		(property "Datasheet" "https://www.onsemi.com/pub/Collateral/2N3903-D.PDF"
-			(at 152.4 67.31 0)
+			(at 215.9 67.31 0)
 			(effects
 				(font
@@
 		)
 		(property "Description" "0.2A Ic, 40V Vce, Small Signal NPN Transistor, TO-92"
-			(at 152.4 67.31 0)
-			(effects
-				(font
+			(at 215.9 67.31 0)
+			(effects
+				(font
