File: 07-brain/electronics/ui/brain-ui.kicad_pcb (KiCad board)
At the start: 2 copper layers, 58 x 110 mm, 30 parts, among them J1 Conn_02x03_Odd_Even, J3 Conn_02x03_Odd_Even, J4 Conn_01x02, J5 Conn_01x06, J6 Conn_02x03_Odd_Even, J8 Conn_02x03_Odd_Even

Commit message: Brain PCB WIP
Parts:
- removed A1: RaspberryPi_Pico, Module:RaspberryPi_Pico_SMD
- removed the G*** at (132.6, 73.0)
- removed the G*** at (130.1, 126.7)
- removed H5, H6: MountingHole, MountingHole:MountingHole_3.2mm_M3_DIN965_Pad
- removed J_TEST_JACK1, J_TEST_JACK2, J_TEST_JACK3, J_TEST_JACK4, J_TEST_JACK5, J_TEST_JACK6, J_TEST_JACK7, J_TEST_JACK8, J_TEST_JACK9: PJ398SM, Shmoergh_Custom_Footprints:Jack_3.5mm_QingPu_WQP-PJ398SM_Vertical_CircularHoles
- removed RV_TEST1, RV_TEST2, RV_TEST3: 100k, Shmoergh_Custom_Footprints:Potentiometer_Bourns_Single-PTV09A
- added D1: LED, LED_THT:LED_D3.0mm, F.Cu at (131.7, 103.0)
- added D2: LED, LED_THT:LED_D3.0mm, F.Cu at (139.7, 103.0)
- added D3: LED, LED_THT:LED_D3.0mm, F.Cu at (147.7, 103.0)
- added D4: LED, LED_THT:LED_D3.0mm, F.Cu at (155.7, 103.0)
- added D5: LED, LED_THT:LED_D3.0mm, F.Cu at (163.7, 103.0)
- added D6: LED, LED_THT:LED_D3.0mm, F.Cu at (171.7, 103.0)
- added J2: Conn_01x02, Connector_PinSocket_2.54mm:PinSocket_1x02_P2.54mm_Vertical, F.Cu at (270.4, 64.7)
- added J7: Conn_02x05_Odd_Even, Connector_PinSocket_2.54mm:PinSocket_2x05_P2.54mm_Vertical, B.Cu at (161.0, 96.5)
- added J_AUDIO_CV_IN1: PJ398SM, Shmoergh_Custom_Footprints:Jack_3.5mm_QingPu_WQP-PJ398SM_Vertical_CircularHoles, F.Cu at (137.0, 115.0)
- added J_AUDIO_CV_IN2: PJ398SM, Shmoergh_Custom_Footprints:Jack_3.5mm_QingPu_WQP-PJ398SM_Vertical_CircularHoles, F.Cu at (153.0, 115.0)
- added J_AUDIO_CV_OUT1: PJ398SM, Shmoergh_Custom_Footprints:Jack_3.5mm_QingPu_WQP-PJ398SM_Vertical_CircularHoles, F.Cu at (137.0, 139.0)
- added J_AUDIO_CV_OUT2: PJ398SM, Shmoergh_Custom_Footprints:Jack_3.5mm_QingPu_WQP-PJ398SM_Vertical_CircularHoles, F.Cu at (153.0, 139.0)
- added J_MIDI1: PJ398SM, Shmoergh_Custom_Footprints:Jack_3.5mm_QingPu_WQP-PJ398SM_Vertical_CircularHoles, F.Cu at (169.0, 83.0)
- added J_PULSE_IN1: PJ398SM, Shmoergh_Custom_Footprints:Jack_3.5mm_QingPu_WQP-PJ398SM_Vertical_CircularHoles, F.Cu at (169.0, 115.0)
- added J_PULSE_OUT1: PJ398SM, Shmoergh_Custom_Footprints:Jack_3.5mm_QingPu_WQP-PJ398SM_Vertical_CircularHoles, F.Cu at (169.0, 139.0)
- added Q1: 2N3904, Package_TO_SOT_THT:TO-92_Inline_Wide, F.Cu at (203.7, 77.4)
- added Q2: 2N3904, Package_TO_SOT_THT:TO-92_Inline_Wide, F.Cu at (203.7, 83.2)
- added Q3: 2N3904, Package_TO_SOT_THT:TO-92_Inline_Wide, F.Cu at (203.7, 88.9)
- added Q4: 2N3904, Package_TO_SOT_THT:TO-92_Inline_Wide, F.Cu at (203.7, 94.7)
- added Q5: 2N3904, Package_TO_SOT_THT:TO-92_Inline_Wide, F.Cu at (203.7, 100.5)
- added Q6: 2N3904, Package_TO_SOT_THT:TO-92_Inline_Wide, F.Cu at (203.7, 106.3)
- added R1: 470, Shmoergh_Custom_Footprints:R_Axial_DIN0207_L6.3mm_D2.5mm_P7.62mm_Horizontal, F.Cu at (255.8, 68.3)
- added R10: 1k, Shmoergh_Custom_Footprints:R_Axial_DIN0207_L6.3mm_D2.5mm_P7.62mm_Horizontal, F.Cu at (224.4, 95.0)
- added R11: 47k, Shmoergh_Custom_Footprints:R_Axial_DIN0207_L6.3mm_D2.5mm_P7.62mm_Horizontal, F.Cu at (228.4, 87.5)
- added R12: 47k, Shmoergh_Custom_Footprints:R_Axial_DIN0207_L6.3mm_D2.5mm_P7.62mm_Horizontal, F.Cu at (228.4, 90.0)
- added R13: 1k, Shmoergh_Custom_Footprints:R_Axial_DIN0207_L6.3mm_D2.5mm_P7.62mm_Horizontal, F.Cu at (228.4, 92.5)
- added R14: 1k, Shmoergh_Custom_Footprints:R_Axial_DIN0207_L6.3mm_D2.5mm_P7.62mm_Horizontal, F.Cu at (228.4, 95.0)
- added R2: 470, Shmoergh_Custom_Footprints:R_Axial_DIN0207_L6.3mm_D2.5mm_P7.62mm_Horizontal, F.Cu at (255.8, 70.8)
- added R3: 47k, Shmoergh_Custom_Footprints:R_Axial_DIN0207_L6.3mm_D2.5mm_P7.62mm_Horizontal, F.Cu at (220.4, 87.5)
- added R4: 47k, Shmoergh_Custom_Footprints:R_Axial_DIN0207_L6.3mm_D2.5mm_P7.62mm_Horizontal, F.Cu at (220.4, 90.0)
- added R5: 1k, Shmoergh_Custom_Footprints:R_Axial_DIN0207_L6.3mm_D2.5mm_P7.62mm_Horizontal, F.Cu at (220.4, 92.5)
- added R6: 1k, Shmoergh_Custom_Footprints:R_Axial_DIN0207_L6.3mm_D2.5mm_P7.62mm_Horizontal, F.Cu at (220.4, 95.0)
- added R7: 47k, Shmoergh_Custom_Footprints:R_Axial_DIN0207_L6.3mm_D2.5mm_P7.62mm_Horizontal, F.Cu at (224.4, 87.5)
- added R8: 47k, Shmoergh_Custom_Footprints:R_Axial_DIN0207_L6.3mm_D2.5mm_P7.62mm_Horizontal, F.Cu at (224.4, 90.0)
- added R9: 1k, Shmoergh_Custom_Footprints:R_Axial_DIN0207_L6.3mm_D2.5mm_P7.62mm_Horizontal, F.Cu at (224.4, 92.5)
- added RV_POT1: 100k, Shmoergh_Custom_Footprints:Potentiometer_Bourns_Single-PTV09A, F.Cu at (137.0, 58.8)
- added RV_POT2: 100k, Shmoergh_Custom_Footprints:Potentiometer_Bourns_Single-PTV09A, F.Cu at (153.0, 58.8)
- added RV_POT3: 100k, Shmoergh_Custom_Footprints:Potentiometer_Bourns_Single-PTV09A, F.Cu at (169.0, 59.0)
- added U_BTN1: SW_SPST_Push_LED, Shmoergh_Custom_Footprints:SPST_Circular_Pushbutton_LED, F.Cu at (137.0, 83.0)
- added U_BTN2: SW_SPST_Push_LED, Shmoergh_Custom_Footprints:SPST_Circular_Pushbutton_LED, F.Cu at (153.0, 83.0)
- J1, J8: moved to F.Cu
- J3: value Conn_02x03_Odd_Even -> Conn_01x02; footprint Connector_PinSocket_2.54mm:PinSocket_2x03_P2.54mm_Vertical -> Connector_PinSocket_2.54mm:PinSocket_1x02_P2.54mm_Vertical; moved to F.Cu
- J4: value Conn_01x02 -> Conn_02x02_Odd_Even; footprint Connector_PinSocket_2.54mm:PinSocket_1x02_P2.54mm_Vertical -> Connector_PinSocket_2.54mm:PinSocket_2x02_P2.54mm_Vertical
- J5: value Conn_01x06 -> Conn_02x03_Odd_Even; footprint Connector_PinSocket_2.54mm:PinSocket_1x06_P2.54mm_Vertical -> Connector_PinSocket_2.54mm:PinSocket_2x03_P2.54mm_Vertical; moved to F.Cu
- J6: value Conn_02x03_Odd_Even -> Conn_02x02_Odd_Even; footprint Connector_PinSocket_2.54mm:PinSocket_2x03_P2.54mm_Vertical -> Connector_PinSocket_2.54mm:PinSocket_2x02_P2.54mm_Vertical; moved to F.Cu
- moved J8 249.9 mm to (270.4, 55.0), turned to 0 degrees
- moved J6 227.3 mm to (256.1, 62.2), turned to 0 degrees
- moved J3 226.0 mm to (275.0, 64.7), turned to 0 degrees
- moved J5 224.8 mm to (263.3, 55.0), turned to 0 degrees
- moved J1 222.4 mm to (265.8, 64.7), turned to 0 degrees
- moved G*** 88.6 mm to (69.4, 103.4)
- moved J4 15.7 mm to (256.1, 55.0)
Connections:
- J3 pad 1: VCA_OUT -> +12V
- J3 pad 2: unconnected-(J3-Pin_2-Pad2) -> +3.3V
- J4 pad 1: GND -> BTN_2
- J4 pad 2: GND -> BTN_LED_1
- J5 pad 1: GATE_DEFAULT -> LED_3
- J5 pad 2: GATE -> LED_4
- J5 pad 3: ENV_OUT_DEFAULT -> LED_2
- J5 pad 4: VCA_IN_DEFAULT -> LED_5
- J5 pad 5: VCA_CV_DEFAULT -> LED_1
- J5 pad 6: VCA_OUT_DEFAULT -> LED_6
- J6 pad 1: LED_A -> MIDI_5T
- J6 pad 2: SUSTAIN_1 -> PULSE_IN
- J6 pad 3: LED_K -> MIDI_4R
- J6 pad 4: SUSTAIN_2 -> PULSE_OUT
- J8 pad 1: GATE -> GND
- J8 pad 2: ATTACK_3 -> AUDIO_CV_OUT_2
- J8 pad 3: RELEASE_1 -> GND
- J8 pad 4: ENV_OUT -> GND
- J8 pad 5: DECAY_1 -> AUDIO_CV_OUT_1
- J8 pad 6: A1_D3_R3 -> GND

Commit message: Designed Brain UI PCB
Parts:
- J1, J3, J4, J5, J6, J8: moved to B.Cu
- moved J8 165.7 mm to (136.0, 152.0), turned to -90 degrees
- moved J3 149.2 mm to (126.0, 57.5), turned to 180 degrees
- moved J2 146.6 mm to (151.7, 150.8), turned to 90 degrees
- moved J1 131.1 mm to (168.0, 152.0), turned to -90 degrees
- moved R1 117.1 mm to (140.9, 90.9), turned to 180 degrees
- moved J6 115.4 mm to (141.5, 49.0)
- moved R2 112.5 mm to (145.1, 90.6), turned to 90 degrees
- moved J4 110.0 mm to (154.0, 96.0)
- moved J5 98.4 mm to (165.0, 49.5), turned to -90 degrees
- moved R5 88.4 mm to (133.1, 106.8)
- moved Q1 81.8 mm to (129.4, 111.7), turned to 90 degrees
- moved R13 80.5 mm to (149.1, 106.8)
- moved R9 79.9 mm to (145.0, 101.8), turned to -90 degrees
- moved R11 78.7 mm to (161.8, 45.6), turned to 180 degrees
- moved Q2 74.7 mm to (129.9, 94.4), turned to -90 degrees
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Connections:
- J4 pad 1: BTN_2 -> BTN_1
- J4 pad 2: BTN_LED_1 -> BTN_LED_2
- J4 pad 3: BTN_1 -> BTN_2
- J4 pad 4: BTN_LED_2 -> BTN_LED_1
- J5 pad 1: LED_3 -> LED_1
- J5 pad 2: LED_4 -> LED_6
- J5 pad 5: LED_1 -> LED_3
- J5 pad 6: LED_6 -> LED_4
- J7 pad 1: POT_3 -> POT_2
- J7 pad 10: AUDIO_CV_IN_1 -> AUDIO_CV_IN_2
- J7 pad 2: GND -> POT_3
- J7 pad 3: POT_2 -> POT_1
- J7 pad 5: POT_1 -> GND
- J7 pad 6: AUDIO_CV_IN_2 -> AUDIO_CV_IN_1
- R10 pad 1: Net-(D4-A) -> Net-(D5-A)
- R11 pad 2: Net-(Q5-B) -> Net-(Q3-B)
- R13 pad 1: Net-(D5-A) -> Net-(D3-A)
- R4 pad 2: Net-(Q2-B) -> Net-(Q4-B)
- R6 pad 1: Net-(D2-A) -> Net-(D4-A)
- R7 pad 2: Net-(Q3-B) -> Net-(Q2-B)
- R8 pad 2: Net-(Q4-B) -> Net-(Q5-B)
- R9 pad 1: Net-(D3-A) -> Net-(D2-A)
Routing:
- net +12V: track 0.00 -> 222.2 mm
- net PULSE_OUT: track 0.00 -> 142.2 mm, vias 0 -> 2
- net PULSE_IN: track 0.00 -> 140.4 mm, vias 0 -> 2
- net Net-(Q1-B): track 0.00 -> 84.9 mm, vias 0 -> 2
- net AUDIO_CV_IN_1: track 0.00 -> 71.3 mm, vias 0 -> 4
- net Net-(Q2-B): track 0.00 -> 66.7 mm, vias 0 -> 2
- net Net-(Q3-B): track 0.00 -> 66.6 mm, vias 0 -> 2
- net MIDI_5T: track 0.00 -> 61.4 mm
- net +3.3V: track 0.00 -> 56.0 mm, vias 0 -> 4
- net MIDI_4R: track 0.00 -> 55.7 mm
- net POT_1: track 0.00 -> 48.4 mm, vias 0 -> 1
- net LED_3: track 0.00 -> 47.1 mm
- net Net-(Q6-B): track 0.00 -> 44.0 mm
- net POT_2: track 0.00 -> 36.5 mm, vias 0 -> 2
- net Net-(D4-K): track 0.00 -> 34.9 mm
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- removed copper zone on F.Cu, net GND

Commit message: Refined Brain PCBs
Parts:
- added G***: LOGO, Shmoergh_Logo:Gyeszno, F.Cu at (178.2, 121.6)
- J_MIDI1: value PJ398SM -> PJ398SM-STEREO
- moved G*** 98.6 mm to (127.9, 140.0), turned to 90 degrees
Changed lines of the file:
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@@
 		(locked yes)
 		(layer "F.Cu")
-		(at 78 55)
+		(at 127.937 140.012 90)
 		(property "Reference" "G***"
-			(at 0 0 0)
+			(at 0 0 90)
 			(layer "F.SilkS")
 			(hide yes)
@@
 		)
 		(property "Value" "LOGO"
-			(at 0.75 0 0)
+			(at 0.75 0 90)
 			(layer "F.SilkS")
 			(hide yes)
@@
 		)
 		(property "Datasheet" ""
-			(at 0 0 0)
+			(at 0 0 90)
 			(layer "F.Fab")
 			(hide yes)
@@
 		)
 		(property "Description" ""
-			(at 0 0 0)
+			(at 0 0 90)
 			(layer "F.Fab")
 			(hide yes)
@@
 			)
 		)
-		(property "Value" "PJ398SM"
+		(property "Value" "PJ398SM-STEREO"
 			(at 0 -1.48 180)
 			(layer "F.Fab")
@@
 		)
 		(embedded_fonts no)
+	)
+	(footprint "Shmoergh_Logo:Gyeszno"
+		(locked yes)
+		(layer "F.Cu")
+		(at 178.229 121.597 -90)
+		(property "Reference" "G***"
+			(at 0 0 90)
+			(layer "F.SilkS")
+			(hide yes)
+			(effects
+				(font
+					(size 1.524 1.524)
+					(thickness 0.3)
+				)
+			)
+		)
+		(property "Value" "LOGO"
+			(at 0.75 0 90)
+			(layer "F.SilkS")
+			(hide yes)
+			(effects
+				(font
+					(size 1.524 1.524)
+					(thickness 0.3)
+				)
+			)
+		)
+		(property "Datasheet" ""
+			(at 0 0 90)
+			(layer "F.Fab")
+			(hide yes)
+			(effects
+				(font
+					(size 1.27 1.27)
+					(thickness 0.15)
+				)
+			)
+		)
+		(property "Description" ""
+			(at 0 0 90)
+			(layer "F.Fab")
+			(hide yes)
+			(effects
+				(font
+					(size 1.27 1.27)
+					(thickness 0.15)
+				)
+			)
+		)
+		(attr through_hole)
+		(fp_poly
+			(pts
+				(xy 2.8702 -2.2606) (xy 2.5527 -2.2606) (xy 2.5527 -2.5654) (xy 2.8702 -2.5654) (xy 2.8702 -2.2606)
+			)
+			(stroke
+				(width 0.01)
+				(type solid)
+			)
+			(fill yes)
+			(layer "F.SilkS")
+		)
+		(fp_poly
+			(pts
+				(xy 2.8702 -2.8702) (xy 3.5052 -2.8702) (xy 3.5052 -2.5654) (xy 2.8702 -2.5654) (xy 2.8702 -2.8702)
+			)
+			(stroke
+				(width 0.01)
+				(type solid)
+			)
+			(fill yes)
+			(layer "F.SilkS")
+		)
+		(fp_poly
+			(pts
+				(xy -1.905 2.2733) (xy -2.2225 2.2733) (xy -2.2225 2.8702) (xy -2.8575 2.8702) (xy -2.8575 2.2733)
+				(xy -2.54 2.2733) (xy -2.54 1.651) (xy -1.905 1.651) (xy -1.905 2.2733)
+			)
+			(stroke
+				(width 0.01)
+				(type solid)
+			)
+			(fill yes)
+			(layer "F.SilkS")
+		)
+		(fp_poly
+			(pts
+				(xy 1.27 2.2733) (xy 0.9525 2.2733) (xy 0.9525 2.5654) (xy 0.635 2.5654) (xy 0.635 2.8702) (xy 0.3175 2.8702)
+				(xy 0.3175 2.2733) (xy 0.635 2.2733) (xy 0.635 1.651) (xy 1.27 1.651) (xy 1.27 2.2733)
+			)
+			(stroke
+				(width 0.01)
+				(type solid)
+			)
+			(fill yes)
+			(layer "F.SilkS")
+		)
+		(fp_poly
+			(pts
+				(xy 1.6002 -2.5654) (xy 2.2352 -2.5654) (xy 2.2352 -2.2098) (xy 2.5527 -2.2098) (xy 2.5527 -1.9685)
+				(xy 2.8702 -1.9685) (xy 2.8702 -1.6637) (xy 3.1877 -1.6637) (xy 3.1877 -1.9685) (xy 3.5052 -1.9685)
+				(xy 3.5052 -2.5654) (xy 3.8227 -2.5654) (xy 3.8227 -2.2606) (xy 4.1402 -2.2606) (xy 4.1402 -2.0193)
+				(xy 3.8227 -2.0193) (xy 3.8227 -1.7145) (xy 3.5052 -1.7145) (xy 3.5052 -1.3716) (xy 3.1877 -1.3716)
+				(xy 3.1877 1.0414) (xy 2.8702 1.0414) (xy 2.8702 2.2733) (xy 2.5527 2.2733) (xy 2.5527 2.5654) (xy 2.2352 2.5654)
+				(xy 2.2352 2.8702) (xy 1.9177 2.8702) (xy 1.9177 1.651) (xy 1.6002 1.651) (xy 1.6002 1.3462) (xy 0.635 1.3462)
+				(xy 0.635 1.651) (xy -0.635 1.651) (xy -0.635 1.9431) (xy -0.9525 1.9431) (xy -0.9525 2.5146) (xy -1.27 2.5146)
+				(xy -1.27 2.8702) (xy -1.5875 2.8702) (xy -1.5875 1.3462) (xy -3.4925 1.3462) (xy -3.4925 1.0414)
+				(xy -4.1275 1.0414) (xy -4.1275 0.1524) (xy -3.81 0.1524) (xy -3.81 -0.1651) (xy -3.4925 -0.1651)
+				(xy -3.175 -0.1651) (xy -3.175 0.1524) (xy -2.8575 0.1524) (xy -2.8575 -0.1651) (xy -2.54 -0.1651)
+				(xy -2.54 0.1524) (xy -2.2225 0.1524) (xy -2.2225 -0.1651) (xy -2.54 -0.1651) (xy -2.8575 -0.1651)
+				(xy -3.175 -0.1651) (xy -3.4925 -0.1651) (xy -3.4925 -1.0668) (xy -4.1275 -1.0668) (xy -4.1275 -1.9685)
+				(xy -3.4925 -1.9685) (xy -3.4925 -1.6637) (xy -2.8575 -1.6637) (xy -2.8575 -1.3716) (xy -2.54 -1.3716)
+				(xy -2.54 -2.2606) (xy -2.2225 -2.2606) (xy -2.2225 -2.5654) (xy -1.5875 -2.5654) (xy -1.5875 -2.8702)
+				(xy 1.6002 -2.8702) (xy 1.6002 -2.5654)
+			)
+			(stroke
+				(width 0.01)
+				(type solid)
+			)
+			(fill yes)
+			(layer "F.SilkS")
+		)
+		(embedded_fonts no)

Commit message: Brain electronics prod ready
Parts:
- added G***: LOGO, Shmoergh_Logo:Gyeszno, B.Cu at (127.9, 138.4)
- moved G*** 96.4 mm to (160.3, 71.3), turned to 180 degrees
- moved G*** 83.5 mm to (137.5, 126.8), turned to 0 degrees
- moved G*** 62.7 mm to (127.6, 77.3)
- moved G*** 20.3 mm to (178.2, 141.9)
Other:
- board text added: "HM-07 BRAIN V0.1 2025 SEP"
- board text removed: "-12V"
- board text removed: "A1/D3/ R3"
- board text removed: "ATTACK 3"
- board text removed: "DEC"
- board text removed: "DEFAULTS"
- board text removed: "ENV"
- board text removed: "ENV OUT"
- board text removed: "GATD"
- board text removed: "GATE"
- board text removed: "GATI"
- board text removed: "HM-05 ADSR VCA V0.2 2025 AUG"
- board text removed: "REL"
- board text removed: "VCIN"
- board text removed: "VCOUT"
- board text removed: "VCV"
