File: 02-vco/electronics/ui-free-tuning/vco-ui.kicad_sch (KiCad schematic)
At the start: 32 parts, among them J1 Conn_01x04, J2 Conn_02x05_Odd_Even, J3 Conn_02x03_Odd_Even, J4 Conn_01x02, J5 Conn_02x02_Counter_Clockwise, J6 Conn_01x06, U1 0203

Commit message: Added VCO output to default connector
Parts:
- J6: value Conn_01x06 -> Conn_01x07; footprint Connector_PinSocket_2.54mm:PinSocket_1x06_P2.54mm_Vertical -> Connector_PinSocket_2.54mm:PinSocket_1x07_P2.54mm_Vertical; symbol Connector_Generic:Conn_01x06 -> Connector_Generic:Conn_01x07
Connections:
- net OUT_DEFAULT: now also J6.7 (Pin_7); no longer J6.6 (Pin_6)
- net OUT_OUT: now reaches J_OUT1.T, U1.1
- net OUT_OUT: now also J6.6 (Pin_6)
Changed lines of the file:
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@@
 		(color 0 0 0 0)
 	)
+	(junction
+		(at 179.07 134.62)
+		(diameter 0)
+		(color 0 0 0 0)
+	)
 	(no_connect
 		(at 229.87 127)
@@
 	(wire
 		(pts
+			(xy 176.53 130.81) (xy 179.07 130.81)
+		)
+		(stroke
+			(width 0)
+			(type default)
+		)
+	)
+	(wire
+		(pts
 			(xy 58.42 67.31) (xy 54.61 67.31)
 		)
@@
 	(wire
 		(pts
-			(xy 152.4 134.62) (xy 180.34 134.62)
+			(xy 152.4 134.62) (xy 179.07 134.62)
 		)
 		(stroke
@@
 	(wire
 		(pts
+			(xy 179.07 134.62) (xy 180.34 134.62)
+		)
+		(stroke
+			(width 0)
+			(type default)
+		)
+	)
+	(wire
+		(pts
 			(xy 252.73 44.45) (xy 250.19 44.45)
 		)
@@
 	(wire
 		(pts
+			(xy 259.08 104.14) (xy 261.62 104.14)
+		)
+		(stroke
+			(width 0)
+			(type default)
+		)
+	)
+	(wire
+		(pts
 			(xy 50.8 139.7) (xy 50.8 142.24)
 		)
@@
 	(wire
 		(pts
+			(xy 179.07 130.81) (xy 179.07 134.62)
+		)
+		(stroke
+			(width 0)
+			(type default)
+		)
+	)
+	(wire
+		(pts
 			(xy 152.4 161.29) (xy 152.4 134.62)
 		)
@@
 		)
 	)
+	(global_label "OUT_OUT"
+		(shape input)
+		(at 176.53 130.81 180)
+		(fields_autoplaced yes)
+		(effects
+			(font
+				(size 1.27 1.27)
+			)
+			(justify right)
+		)
+		(property "Intersheetrefs" "${INTERSHEET_REFS}"
+			(at 165.32 130.81 0)
+			(effects
+				(font
+					(size 1.27 1.27)
+				)
+				(justify right)
+				(hide yes)
+			)
+		)
+	)
 	(global_label "PWM_DEFAULT"
 		(shape output)
@@
 	(global_label "OUT_DEFAULT"
 		(shape output)
-		(at 259.08 101.6 180)
+		(at 259.08 104.14 180)
 		(fields_autoplaced yes)
 		(effects
@@
 		)
 		(property "Intersheetrefs" "${INTERSHEET_REFS}"
-			(at 243.5762 101.6 0)
+			(at 243.5762 104.14 0)
 			(effects
 				(font
@@
 		)
 	)
+	(global_label "OUT_OUT"
+		(shape output)
+		(at 259.08 101.6 180)
+		(fields_autoplaced yes)
+		(effects
+			(font
+				(size 1.27 1.27)
+			)
+			(justify right)
+		)
+		(property "Intersheetrefs" "${INTERSHEET_REFS}"
+			(at 247.87 101.6 0)
+			(effects
+				(font
+					(size 1.27 1.27)
+				)
+				(justify right)
+				(hide yes)
+			)
+		)
+	)
 	(global_label "FM_DEFAULT"
 		(shape output)
@@
 	)
 	(symbol
-		(lib_id "Connector_Generic:Conn_01x06")
-		(at 266.7 93.98 0)
+		(lib_id "Connector_Generic:Conn_01x07")
+		(at 266.7 96.52 0)
 		(unit 1)
 		(exclude_from_sim no)
@@
 		(fields_autoplaced yes)
 		(property "Reference" "J6"
-			(at 269.24 93.9799 0)
+			(at 269.24 95.2499 0)
 			(effects
 				(font
@@
 			)
 		)
-		(property "Value" "Conn_01x06"
-			(at 269.24 96.5199 0)
+		(property "Value" "Conn_01x07"
+			(at 269.24 97.7899 0)
 			(effects
 				(font
@@
 			)
 		)
-		(property "Footprint" "Connector_PinSocket_2.54mm:PinSocket_1x06_P2.54mm_Vertical"
-			(at 266.7 93.98 0)
+		(property "Footprint" "Connector_PinSocket_2.54mm:PinSocket_1x07_P2.54mm_Vertical"
+			(at 266.7 96.52 0)
 			(effects
 				(font
@@
 		)
 		(property "Datasheet" "~"
-			(at 266.7 93.98 0)
+			(at 266.7 96.52 0)
 			(effects
 				(font
@@
 			)
 		)
-		(property "Description" "Generic connector, single row, 01x06, script generated (kicad-library-utils/schlib/autogen/connector/)"
-			(at 266.7 93.98 0)
+		(property "Description" "Generic connector, single row, 01x07, script generated (kicad-library-utils/schlib/autogen/connector/)"
+			(at 266.7 96.52 0)
 			(effects
 				(font
@@
 		)
 		(property "Part URL" "https://mou.sr/4lnf48h"
-			(at 266.7 93.98 0)
+			(at 266.7 96.52 0)
 			(effects
 				(font
@@
 		)
 		(property "Vendor" "Mouser"
-			(at 266.7 93.98 0)
+			(at 266.7 96.52 0)
 			(effects
 				(font
@@
 		)
 		(property "LCSC" ""
-			(at 266.7 93.98 0)
+			(at 266.7 96.52 0)
 			(effects
 				(font
@@
 		)
 		(property "Part no." "200-SSW10601TS"
-			(at 266.7 93.98 0)
+			(at 266.7 96.52 0)
+			(effects
+				(font
+					(size 1.27 1.27)
+				)
+				(hide yes)
+			)
+		)
+		(property "Part No." ""
+			(at 266.7 96.52 0)
 			(effects
 				(font
@@
 		(pin "5"
 		)
+		(pin "7"
+		)
 		(instances

Commit message: Added CV output to VCO default patch
Connections:
- net CV_INPUT: now reaches J_CV1.T, R3.1
- net CV_INPUT: now also J6.6 (Pin_6)
- net OUT_OUT: no longer names the net of J_OUT1.T, U1.1
- net OUT_OUT: no longer J6.6 (Pin_6)
Changed lines of the file:
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@@
+	)
+	(junction
+		(at 57.15 134.62)
+		(diameter 0)
+		(color 0 0 0 0)
 	)
 	(junction
@@
 		(color 0 0 0 0)
 	)
-	(junction
-		(at 179.07 134.62)
-		(diameter 0)
-		(color 0 0 0 0)
-	)
 	(no_connect
 		(at 229.87 127)
@@
 	(wire
 		(pts
-			(xy 176.53 130.81) (xy 179.07 130.81)
-		)
-		(stroke
-			(width 0)
-			(type default)
-		)
-	)
-	(wire
-		(pts
 			(xy 58.42 67.31) (xy 54.61 67.31)
 		)
@@
 	(wire
 		(pts
-			(xy 152.4 134.62) (xy 179.07 134.62)
-		)
-		(stroke
-			(width 0)
-			(type default)
-		)
-	)
-	(wire
-		(pts
 			(xy 104.14 125.73) (xy 104.14 128.27)
 		)
@@
 	(wire
 		(pts
-			(xy 179.07 134.62) (xy 180.34 134.62)
+			(xy 152.4 134.62) (xy 180.34 134.62)
+		)
+		(stroke
+			(width 0)
+			(type default)
+		)
+	)
+	(wire
+		(pts
+			(xy 57.15 134.62) (xy 55.88 134.62)
 		)
 		(stroke
@@
 	(wire
 		(pts
-			(xy 59.69 134.62) (xy 55.88 134.62)
+			(xy 59.69 134.62) (xy 57.15 134.62)
 		)
 		(stroke
@@
 	(wire
 		(pts
+			(xy 57.15 123.19) (xy 57.15 134.62)
+		)
+		(stroke
+			(width 0)
+			(type default)
+		)
+	)
+	(wire
+		(pts
 			(xy 165.1 107.95) (xy 165.1 110.49)
 		)
@@
 	(wire
 		(pts
+			(xy 62.23 123.19) (xy 57.15 123.19)
+		)
+		(stroke
+			(width 0)
+			(type default)
+		)
+	)
+	(wire
+		(pts
 			(xy 50.8 107.95) (xy 50.8 110.49)
 		)
@@
 		(pts
 			(xy 220.98 52.07) (xy 220.98 46.99)
-		)
-		(stroke
-			(width 0)
-			(type default)
-		)
-	)
-	(wire
-		(pts
-			(xy 179.07 130.81) (xy 179.07 134.62)
 		)
 		(stroke
@@
 		)
 	)
+	(global_label "CV_INPUT"
+		(shape output)
+		(at 62.23 123.19 0)
+		(fields_autoplaced yes)
+		(effects
+			(font
+				(size 1.27 1.27)
+			)
+			(justify left)
+		)
+		(property "Intersheetrefs" "${INTERSHEET_REFS}"
+			(at 74.0448 123.19 0)
+			(effects
+				(font
+					(size 1.27 1.27)
+				)
+				(justify left)
+				(hide yes)
+			)
+		)
+	)
 	(global_label "FM_DEFAULT"
 		(shape input)
@@
 		)
 	)
-	(global_label "OUT_OUT"
-		(shape input)
-		(at 176.53 130.81 180)
-		(fields_autoplaced yes)
-		(effects
-			(font
-				(size 1.27 1.27)
-			)
-			(justify right)
-		)
-		(property "Intersheetrefs" "${INTERSHEET_REFS}"
-			(at 165.32 130.81 0)
-			(effects
-				(font
-					(size 1.27 1.27)
-				)
-				(justify right)
-				(hide yes)
-			)
-		)
-	)
 	(global_label "PWM_DEFAULT"
 		(shape output)
@@
 		)
 	)
-	(global_label "OUT_OUT"
+	(global_label "CV_INPUT"
 		(shape output)
 		(at 259.08 101.6 180)
@@
 		)
 		(property "Intersheetrefs" "${INTERSHEET_REFS}"
-			(at 247.87 101.6 0)
-			(effects
-				(font
+			(at 247.2652 101.6 0)
+			(effects
+				(font
