File: 07-brain/electronics/v0.2/core/sheets/pots.kicad_sch (KiCad schematic)
At the start: 3 parts, among them U10 74HC4051

Commit message: Removed one pot and added one button in Brain
Connections:
- net POT_3 is gone; now on net GND: U10.15 (A2)
Changed lines of the file:
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@@
+	)
+	(junction
+		(at 121.92 76.2)
+		(diameter 0)
+		(color 0 0 0 0)
 	)
 	(junction
@@
 	(wire
 		(pts
-			(xy 110.49 130.81) (xy 96.52 130.81)
-		)
-		(stroke
-			(width 0)
-			(type default)
-		)
-	)
-	(wire
-		(pts
 			(xy 96.52 68.58) (xy 125.73 68.58)
 		)
@@
 	(wire
 		(pts
+			(xy 125.73 73.66) (xy 121.92 73.66)
+		)
+		(stroke
+			(width 0)
+			(type default)
+		)
+	)
+	(wire
+		(pts
 			(xy 135.89 91.44) (xy 135.89 92.71)
 		)
@@
 	(wire
 		(pts
+			(xy 121.92 73.66) (xy 121.92 76.2)
+		)
+		(stroke
+			(width 0)
+			(type default)
+		)
+	)
+	(wire
+		(pts
 			(xy 135.89 40.64) (xy 135.89 63.5)
 		)
@@
 	(wire
 		(pts
-			(xy 110.49 73.66) (xy 110.49 130.81)
-		)
-		(stroke
-			(width 0)
-			(type default)
-		)
-	)
-	(wire
-		(pts
 			(xy 147.32 92.71) (xy 135.89 92.71)
 		)
@@
 	(wire
 		(pts
-			(xy 125.73 73.66) (xy 110.49 73.66)
-		)
-		(stroke
-			(width 0)
-			(type default)
-		)
-	)
-	(wire
-		(pts
 			(xy 67.31 62.23) (xy 67.31 64.77)
 		)
@@
 		)
 	)
-	(hierarchical_label "POT_3"
-		(shape input)
-		(at 96.52 130.81 180)
-		(effects
-			(font
-				(size 1.27 1.27)
-			)
-			(justify right)
-		)
-	)
