File: 07-brain/electronics/v0.2/core/sheets/midi-in.kicad_sch (KiCad schematic)
At the start: 8 parts, among them Q6 MMBT3904, Q7 MMBT3904, U2 6N137

Commit message: Updated pull-up for MIDI opto in v0.2 Brain
Parts:
- R7: value 10k -> 3.3k; LCSC C25804 -> C22978
Changed lines of the file:
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@@
 			)
 		)
-		(property "Value" "10k"
+		(property "Value" "3.3k"
 			(at 170.18 83.82 0)
 			(effects
@@
 			)
 		)
-		(property "LCSC" "C25804"
+		(property "LCSC" "C22978"
 			(at 166.37 85.09 90)
 			(effects
