File: 04-vcf/electronics/ui/vcf-ui.kicad_pcb (KiCad board)
At the start: 2 copper layers, 58 x 110 mm, 46 parts, among them J1 Conn_02x03_Odd_Even, J2 Conn_02x02_Counter_Clockwise, J4 Conn_01x02, J5 Conn_01x06, J6 Conn_02x04_Odd_Even, U1 TL072

Commit message: Fixed VCF v0.1 bugs - new version: v0.2
Other:
- board text added: "+12V"
- board text added: "-12V"
- board text added: "CUTOFF"
- board text added: "CUTOFF POT RANGE"
- board text added: "GND"
- board text added: "HM-04 VCF UI V0.2 2025 JULY"
- board text removed: "HM-04 VCF UI V0.1 2025 JULY"
Changed lines of the file:
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@@
 		(tags "Through hole pin header THT 1x03 2.54mm single row")
 		(property "Reference" "JP1"
-			(at 0 -2.38 0)
+			(at -4.445 6.731 90)
 			(layer "F.SilkS")
 			(effects
@@
 	)
 	(footprint "Shmoergh_Logo:Gyeszno"
-		(locked yes)
 		(layer "F.Cu")
 		(at 147.829 129.979)
@@
 		(embedded_fonts no)
 	)
+	(gr_line
+		(start 128.953 95.816)
+		(end 126.413 95.816)
+		(stroke
+			(width 0.1)
+			(type default)
+		)
+		(layer "F.SilkS")
+	)
+	(gr_line
+		(start 130.858 94.419)
+		(end 129.461 96.324)
+		(stroke
+			(width 0.1)
+			(type default)
+		)
+		(layer "F.SilkS")
+	)
+	(gr_line
+		(start 130.858 93.149)
+		(end 128.953 95.816)
+		(stroke
+			(width 0.1)
+			(type default)
+		)
+		(layer "F.SilkS")
+	)
+	(gr_rect
+		(start 168.577 92.641)
+		(end 173.911 100.388)
+		(stroke
+			(width 0.1)
+			(type default)
+		)
+		(fill no)
+		(layer "F.SilkS")
+	)
 	(gr_rect
 		(start 142.829 144.479)
@@
 		)
 		(fill yes)
-		(locked yes)
 		(layer "F.SilkS")
 	)
@@
 			(type default)
 		)
-		(locked yes)
+		(layer "F.SilkS")
+	)
+	(gr_rect
+		(start 168.577 147.124)
+		(end 173.911 152.331)
+		(stroke
+			(width 0.1)
+			(type default)
+		)
+		(fill no)
 		(layer "F.SilkS")
 	)
@@
 		)
 		(fill yes)
-		(locked yes)
 		(layer "F.SilkS")
 	)
@@
 		)
 		(fill no)
-		(locked yes)
+		(layer "F.SilkS")
+	)
+	(gr_rect
+		(start 131.112 149.537)
+		(end 146.479 152.331)
+		(stroke
+			(width 0.1)
+			(type default)
+		)
+		(fill no)
+		(layer "F.SilkS")
+	)
+	(gr_line
+		(start 126.413 95.816)
+		(end 126.413 96.324)
+		(stroke
+			(width 0.1)
+			(type default)
+		)
 		(layer "F.SilkS")
 	)
@@
 		)
 		(fill yes)
-		(locked yes)
+		(layer "F.SilkS")
+	)
+	(gr_rect
+		(start 125.016 96.578)
+		(end 135.43 101.912)
+		(stroke
+			(width 0.1)
+			(type default)
+		)
+		(fill no)
 		(layer "F.SilkS")
 	)
@@
 	)
 	(gr_text "SHMØERGH \nHOG MODULEUR"
-		(locked yes)
 		(at 143.329 138.979 0)
 		(layer "F.SilkS")
@@
 		)
 	)
+	(gr_text "GND"
+		(at 155.115 62.542 0)
+		(layer "F.SilkS")
+		(effects
+			(font
+				(size 1 0.75)
+				(thickness 0.17)
+				(bold yes)
+			)
+			(justify left bottom)
+		)
+	)
 	(gr_text "DEFAULTS"
 		(at 138.986 148.775 0)
@@
 		)
 	)
+	(gr_text "CUTOFF"
+		(at 130.858 93.657 0)
+		(layer "F.SilkS")
+		(effects
+			(font
+				(size 1 0.75)
+				(thickness 0.17)
+				(bold yes)
+			)
+			(justify left bottom)
+		)
+	)
 	(gr_text "RESO_VALUE"
 		(at 167.688 151.823 0)
@@
 		)
 	)
+	(gr_text "HP"
+		(at 130.858 94.927 0)
+		(layer "F.SilkS")
+		(effects
+			(font
+				(size 1 0.75)
+				(thickness 0.17)
+				(bold yes)
+			)
+			(justify left bottom)
+		)
+	)
+	(gr_text "+12V"
+		(at 170.609 104.96 90)
+		(layer "F.SilkS" knockout)
+		(effects
+			(font
+				(size 1 1)
+				(thickness 0.2)
+				(bold yes)
+			)
+			(justify left bottom)
+		)
+	)
 	(gr_text "NC"
 		(at 145.209 153.728 0)
@@
 		)
 	)
+	(gr_text "+12V"
+		(at 171.244 92.387 0)
+		(layer "F.SilkS")
+		(effects
+			(font
+				(size 1 1)
+				(thickness 0.2)
+				(bold yes)
+			)
+			(justify left bottom)
+		)
+	)
 	(gr_text "BIAS"
 		(at 181.531 68.638 90)
@@
 		)
 	)
+	(gr_text "-12V"
+		(at 154.607 52.255 0)
+		(layer "F.SilkS")
+		(effects
+			(font
+				(size 1 0.75)
+				(thickness 0.17)
+				(bold yes)
+			)
+			(justify left bottom)
+		)
+	)
+	(gr_text "LP"
+		(at 130.858 96.324 0)
+		(layer "F.SilkS")
+		(effects
+			(font
+				(size 1 0.75)
+				(thickness 0.17)
+				(bold yes)
+			)
+			(justify left bottom)
+		)
+	)
+	(gr_text "CUTOFF POT RANGE"
+		(at 154.226 62.669 90)
+		(layer "F.SilkS")
+		(effects
+			(font
+				(size 1 0.75)
+				(thickness 0.17)
+				(bold yes)
+			)
+			(justify left bottom)
+		)
+	)
+	(gr_text "OUT"
+		(at 132.89 103.436 0)
+		(layer "F.SilkS")
+		(effects
+			(font
+				(size 1 0.75)
+				(thickness 0.17)
+				(bold yes)
+			)
+			(justify left bottom)
+		)
+	)
 	(gr_text "HP"
 		(at 132.509 153.728 0)
@@
 		)
 	)
-	(gr_text "HM-04 VCF UI \nV0.1 2025 JULY"
-		(locked yes)
+	(gr_text "HM-04 VCF UI \nV0.2 2025 JULY"
 		(at 143.329 143.479 0)
 		(layer "F.SilkS")
@@
 			(justify left bottom)
 		)
-		(render_cache "HM-04 VCF UI \nV0.1 2025 JULY" 0
+		(render_cache "HM-04 VCF UI \nV0.2 2025 JULY" 0
 			(polygon
 				(pts
@@
 			(polygon
 				(pts
-					(xy 146.838656 142.40533) (xy 146.838656 143.137161) (xy 146.54591 143.137161) (xy 146.54591 143.2835)
-					(xy 147.277741 143.2835) (xy 147.277741 143.137161) (xy 146.984994 143.137161) (xy 146.984994 142.112584)
-					(xy 146.838656 142.112584) (xy 146.838656 142.258992) (xy 146.54591 142.258992) (xy 146.54591 142.40533)
+					(xy 146.54591 142.990823) (xy 146.54591 143.2835) (xy 147.277741 143.2835) (xy 147.277741 143.137161)
+					(xy 146.692248 143.137161) (xy 146.692248 142.990823)
+				)
+			)
+			(polygon
+				(pts
+					(xy 147.131332 142.258992) (xy 147.131332 142.112584) (xy 146.692248 142.112584) (xy 146.692248 142.258992)
+				)
+			)
+			(polygon
+				(pts
+					(xy 147.131332 142.258992) (xy 147.131332 142.551739) (xy 147.277741 142.551739) (xy 147.277741 142.258992)
+				)
+			)
+			(polygon
+				(pts
+					(xy 146.692248 142.844415) (xy 146.692248 142.990823) (xy 146.838656 142.990823) (xy 146.838656 142.844415)
+				)
+			)
+			(polygon
+				(pts
+					(xy 146.54591 142.258992) (xy 146.54591 142.40533) (xy 146.692248 142.40533) (xy 146.692248 142.258992)
+				)
+			)
+			(polygon
+				(pts
+					(xy 146.984994 142.551739) (xy 146.984994 142.698077) (xy 147.131332 142.698077) (xy 147.131332 142.551739)
+				)
+			)
+			(polygon
+				(pts
+					(xy 146.838656 142.698077) (xy 146.838656 142.844415) (xy 146.984994 142.844415) (xy 146.984994 142.698077)
 				)
 			)
@@
 	)
 	(group ""
-		(locked yes)
 		(members "03af84ad-dc1f-45b0-affd-311cb928f7e8" "20fb748d-bea1-42e1-beed-2f4d709fae46"
 			"6606bfb2-6cd3-4d71-b816-d8bd1a09c69f" "9699c592-13f2-4dc9-9f25-f7ce87be5d14"
@@
 	)
 	(group ""
-		(locked yes)
 		(members "6a606e63-46eb-465b-a7da-88840621c518" "f4a4fb2a-cda5-4eba-b4f9-ab9f52153dc4")
 	)
