File: 08-default-patch/default-patch.kicad_sch (KiCad schematic)
At the start: 7 parts

Commit message: Added Default patch PCB
Parts:
- removed J_ENV_VCA1, J_ENV_VCA2, J_FILTER1, J_UTILS_OUT1, J_VCO1, J_VCO2: Conn_01x06, symbol Connector_Generic:Conn_01x06
- added H1, H2, H3, H4: MountingHole, MountingHole:MountingHole_3.2mm_M3, symbol Mechanical:MountingHole
- added JP1, JP10, JP11, JP12, JP13, JP2, JP3, JP4, JP5, JP6, JP7, JP8, JP9: Jumper_2_Bridged, Jumper:SolderJumper-2_P1.3mm_Bridged_RoundedPad1.0x1.5mm, symbol Jumper:Jumper_2_Bridged
- added J_ENV_VCA1, J_ENV_VCA2, J_FILTER1, J_UTILS_OUT1: Conn_01x06, Connector_PinHeader_2.54mm:PinHeader_2x06_P2.54mm_Vertical, symbol Connector_Generic:Conn_02x06_Odd_Even
- added J_VCO1, J_VCO2: Conn_01x07, Connector_PinHeader_2.54mm:PinHeader_2x07_P2.54mm_Vertical, symbol Connector_Generic:Conn_02x07_Odd_Even
- J_MIXER1: footprint (none) -> Connector_PinHeader_2.54mm:PinHeader_2x06_P2.54mm_Vertical; symbol Connector_Generic:Conn_01x06 -> Connector_Generic:Conn_02x06_Odd_Even
Connections:
- net at J_MIXER1.3 (Pin_3): now also J_MIXER1.4 (Pin_4), JP5.2 (B)
- net at J_MIXER1.1 (Pin_1): now also J_MIXER1.2 (Pin_2), JP3.2 (B)
- net at J_MIXER1.5 (Pin_5): now also J_MIXER1.6 (Pin_6), JP4.2 (B)
- new net: JP5.1 (A), J_VCO2.13 (Pin_13), J_VCO2.14 (Pin_14)
- new net: JP4.1 (A), J_VCO1.10 (Pin_10), J_VCO1.9 (Pin_9)
- new net: JP9.1 (A), J_ENV_VCA2.5 (Pin_5), J_ENV_VCA2.6 (Pin_6)
- new net: JP9.2 (B), J_FILTER1.7 (Pin_7), J_FILTER1.8 (Pin_8)
- new net: JP12.1 (A), J_ENV_VCA1.1 (Pin_1), J_ENV_VCA1.2 (Pin_2)
- new net: JP12.2 (B), J_ENV_VCA2.3 (Pin_3), J_ENV_VCA2.4 (Pin_4)
- new net: JP10.1 (A), J_ENV_VCA1.7 (Pin_7), J_ENV_VCA1.8 (Pin_8)
- new net: JP10.2 (B), J_FILTER1.10 (Pin_10), J_FILTER1.9 (Pin_9)
- new net: JP11.1 (A), J_ENV_VCA1.11 (Pin_11), J_ENV_VCA1.12 (Pin_12)
- new net: JP11.2 (B), J_UTILS_OUT1.7 (Pin_7), J_UTILS_OUT1.8 (Pin_8)
- new net: JP1.1 (A), J_VCO1.11 (Pin_11), J_VCO1.12 (Pin_12)
- new net: JP1.2 (B), J_VCO2.7 (Pin_7), J_VCO2.8 (Pin_8)
- new net: JP13.1 (A), J_ENV_VCA1.3 (Pin_3), J_ENV_VCA1.4 (Pin_4)
- new net: JP13.2 (B), J_ENV_VCA2.1 (Pin_1), J_ENV_VCA2.2 (Pin_2)
- new net: JP8.1 (A), J_UTILS_OUT1.11 (Pin_11), J_UTILS_OUT1.12 (Pin_12)
- new net: JP8.2 (B), J_FILTER1.5 (Pin_5), J_FILTER1.6 (Pin_6)
- new net: J_ENV_VCA2.10 (Pin_10), J_ENV_VCA2.9 (Pin_9)
- new net: J_ENV_VCA2.11 (Pin_11), J_ENV_VCA2.12 (Pin_12)
- new net: J_ENV_VCA2.7 (Pin_7), J_ENV_VCA2.8 (Pin_8)
- new net: JP6.1 (A), J_VCO2.10 (Pin_10), J_VCO2.9 (Pin_9)
- new net: JP6.2 (B), J_MIXER1.7 (Pin_7), J_MIXER1.8 (Pin_8)
- new net: JP7.1 (A), J_MIXER1.10 (Pin_10), J_MIXER1.9 (Pin_9)
- new net: JP7.2 (B), J_FILTER1.3 (Pin_3), J_FILTER1.4 (Pin_4)
- new net: JP2.1 (A), J_VCO1.7 (Pin_7), J_VCO1.8 (Pin_8)
- new net: JP2.2 (B), J_VCO2.11 (Pin_11), J_VCO2.12 (Pin_12)
- new net: J_ENV_VCA1.10 (Pin_10), J_ENV_VCA1.9 (Pin_9)
- new net: J_ENV_VCA1.5 (Pin_5), J_ENV_VCA1.6 (Pin_6)
- new net: JP3.1 (A), J_VCO1.13 (Pin_13), J_VCO1.14 (Pin_14)
- new net: J_MIXER1.11 (Pin_11), J_MIXER1.12 (Pin_12)
- new net: J_FILTER1.1 (Pin_1), J_FILTER1.2 (Pin_2)
- new net: J_FILTER1.11 (Pin_11), J_FILTER1.12 (Pin_12)
- new net: J_UTILS_OUT1.1 (Pin_1), J_UTILS_OUT1.2 (Pin_2)
- new net: J_UTILS_OUT1.10 (Pin_10), J_UTILS_OUT1.9 (Pin_9)
- new net: J_UTILS_OUT1.3 (Pin_3), J_UTILS_OUT1.4 (Pin_4)
- new net: J_UTILS_OUT1.5 (Pin_5), J_UTILS_OUT1.6 (Pin_6)
- new net: J_VCO2.1 (Pin_1), J_VCO2.2 (Pin_2)
- new net: J_VCO2.3 (Pin_3), J_VCO2.4 (Pin_4)
- new net: J_VCO2.5 (Pin_5), J_VCO2.6 (Pin_6)
- new net: J_VCO1.1 (Pin_1), J_VCO1.2 (Pin_2)
- new net: J_VCO1.3 (Pin_3), J_VCO1.4 (Pin_4)
- new net: J_VCO1.5 (Pin_5), J_VCO1.6 (Pin_6)
Other:
- note removed: "TODO: VCO default patches here are outdated. Doublecheck the actual VCO schematic and upated the default patch."
