File: 07-brain/electronics/v0.2/ui/sheets/leds.kicad_sch (KiCad schematic)
At the start: 24 parts, among them Q1 2N3904, Q2 2N3904, Q3 2N3904, Q4 2N3904, Q5 2N3904, Q6 2N3904

Commit message: Updated pull-up for MIDI opto in v0.2 Brain
Parts:
- R10, R13, R14, R5, R6, R9: value 1k -> 4.7k
Changed lines of the file:
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@@
 			)
 		)
-		(property "Value" "1k"
+		(property "Value" "4.7k"
 			(at 158.75 44.45 0)
 			(effects
@@
 			)
 		)
-		(property "Value" "1k"
+		(property "Value" "4.7k"
 			(at 158.75 107.95 0)
 			(effects
@@
 			)
 		)
-		(property "Value" "1k"
+		(property "Value" "4.7k"
 			(at 222.25 44.45 0)
 			(effects
@@
 			)
 		)
-		(property "Value" "1k"
+		(property "Value" "4.7k"
 			(at 95.25 44.45 0)
 			(effects
@@
 			)
 		)
-		(property "Value" "1k"
+		(property "Value" "4.7k"
 			(at 95.25 107.95 0)
 			(effects
@@
 			)
 		)
-		(property "Value" "1k"
+		(property "Value" "4.7k"
 			(at 222.25 107.95 0)
 			(effects
